File: MCU Datalogger with built-in EEPROM and clock.kicad_pcb (KiCad board)
At the start: 2 copper layers, 56 x 36 mm, 29 parts, among them J1 Conn_01x04_Pin, J2 Conn_01x09_Pin, J3 Conn_01x04_Pin, J4 Conn_02x03_Odd_Even, U1 DS1337S_, U2 24LC1025, U3 24LC1025, U4 ATMEGA328P-AU, Y1 32.768 kHz, Y2 16MHz

Commit message: Completed 4-layer PCB routing
Parts:
- moved R6 6.11 mm to (145.7, 54.4), turned to 180 degrees
- moved R7 5.93 mm to (150.6, 57.9)
- moved J2 3.56 mm to (116.1, 75.7)
- moved Y2 1.28 mm to (133.3, 69.3)
- moved C1 0.76 mm to (129.3, 50.0)
- moved C3 0.76 mm to (133.7, 50.0)
- moved C5 0.76 mm to (137.7, 50.0)
- moved R1 0.72 mm to (118.3, 70.6)
- moved R2 0.72 mm to (122.8, 70.6)
- moved D1 0.51 mm to (149.9, 50.0)
- moved D2 0.51 mm to (144.5, 50.0)
- moved R5 0.27 mm to (150.4, 54.4), turned to 180 degrees
- turned R4 to 180 degrees
Routing:
- net VCC: track 101.7 -> 54.7 mm, vias 5 -> 10
- net GND: track 60.2 -> 38.3 mm, vias 10 -> 11
- net /D2: track 46.4 -> 31.6 mm, vias 1 -> 0
- net /TX: track 32.9 -> 42.9 mm, vias 1 -> 0
- net /RX: track 30.1 -> 39.3 mm, vias 1 -> 0
- net Net-(U4-PB6): track 28.1 -> 20.9 mm, vias 0 -> 4
- net /RESET: track 26.3 -> 33.5 mm, vias 4 -> 1
- net /D8: track 12.6 -> 17.9 mm, vias 1 -> 0
- net Net-(D2-K): track 9.44 -> 4.79 mm
- net /D5: track 14.4 -> 17.8 mm, vias 1 -> 0
- net /D7: track 13.1 -> 16.5 mm, vias 1 -> 0
- net /D6: track 13.7 -> 16.9 mm, vias 1 -> 0
- net /MOSI: track 28.0 -> 30.9 mm
- net Net-(U4-PB7): track 22.3 -> 24.8 mm, vias 0 -> 4
- net /D3: track 25.0 -> 27.3 mm, vias 1 -> 0
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- added copper zone on In2.Cu, net VCC
- removed copper zone on F.Cu, net VCC
Other:
- copper layers 2 -> 4
